Commit message: Update mac_car

File: mac_car/v6_description/urdf/v6.xacro (robot description, xacro)
@@ -13,5 +13,5 @@
     <origin rpy="0 0 0" xyz="0 0 0"/>
     <geometry>
-      <mesh filename="package://v6_description/meshes/base_link.stl" scale="0.001 0.001 0.001"/>
+      <mesh filename="v6_description/meshes/base_link.stl" scale="0.001 0.001 0.001"/>
     </geometry>
     <material name="silver"/>
@@ -20,5 +20,5 @@
     <origin rpy="0 0 0" xyz="0 0 0"/>
     <geometry>
-      <mesh filename="package://v6_description/meshes/base_link.stl" scale="0.001 0.001 0.001"/>
+      <mesh filename="v6_description/meshes/base_link.stl" scale="0.001 0.001 0.001"/>
     </geometry>
   </collision>
@@ -33,5 +33,5 @@
     <origin rpy="0 0 0" xyz="0.114065 -0.334351 -0.110913"/>
     <geometry>
-      <mesh filename="package://v6_description/meshes/upper_blue_v1_1.stl" scale="0.001 0.001 0.001"/>
+      <mesh filename="v6_description/meshes/upper_blue_v1_1.stl" scale="0.001 0.001 0.001"/>
     </geometry>
     <material name="silver"/>
@@ -40,5 +40,5 @@
     <origin rpy="0 0 0" xyz="0.114065 -0.334351 -0.110913"/>
     <geometry>
-      <mesh filename="package://v6_description/meshes/upper_blue_v1_1.stl" scale="0.001 0.001 0.001"/>
+      <mesh filename="v6_description/meshes/upper_blue_v1_1.stl" scale="0.001 0.001 0.001"/>
     </geometry>
   </collision>
@@ -46,12 +46,12 @@
 <link name="upper_silver_v1_1">
   <inertial>
-    <origin rpy="0 0 0" xyz="-0.05397145103461684 0.12865565118005895 0.06340297559246169"/>
-    <mass value="0.5824308278195107"/>
-    <inertia ixx="0.00486" ixy="0.0" ixz="2.4e-05" iyy="0.001444" iyz="-0.0" izz="0.004712"/>
+    <origin rpy="0 0 0" xyz="-0.05442619134290837 0.1286556607713099 0.06371666752539593"/>
+    <mass value="0.5901067825147455"/>
+    <inertia ixx="0.004878" ixy="0.0" ixz="3e-05" iyy="0.001458" iyz="-0.0" izz="0.004735"/>
   </inertial>
   <visual>
     <origin rpy="0 0 0" xyz="-0.020935 -0.20677 -0.110239"/>
     <geometry>
-      <mesh filename="package://v6_description/meshes/upper_silver_v1_1.stl" scale="0.001 0.001 0.001"/>
+      <mesh filename="v6_description/meshes/upper_silver_v1_1.stl" scale="0.001 0.001 0.001"/>
     </geometry>
     <material name="silver"/>
@@ -60,5 +60,5 @@
     <origin rpy="0 0 0" xyz="-0.020935 -0.20677 -0.110239"/>
     <geometry>
-      <mesh filename="package://v6_description/meshes/upper_silver_v1_1.stl" scale="0.001 0.001 0.001"/>
+      <mesh filename="v6_description/meshes/upper_silver_v1_1.stl" scale="0.001 0.001 0.001"/>
     </geometry>
   </collision>
@@ -73,5 +73,5 @@
     <origin rpy="0 0 0" xyz="0.264049 -0.334351 -0.074934"/>
     <geometry>
-      <mesh filename="package://v6_description/meshes/Side_U_Bracket_Component1_v2_1.stl" scale="0.001 0.001 0.001"/>
+      <mesh filename="v6_description/meshes/Side_U_Bracket_Component1_v2_1.stl" scale="0.001 0.001 0.001"/>
     </geometry>
     <material name="silver"/>
@@ -80,5 +80,5 @@
     <origin rpy="0 0 0" xyz="0.264049 -0.334351 -0.074934"/>
     <geometry>
-      <mesh filename="package://v6_description/meshes/Side_U_Bracket_Component1_v2_1.stl" scale="0.001 0.001 0.001"/>
+      <mesh filename="v6_description/meshes/Side_U_Bracket_Component1_v2_1.stl" scale="0.001 0.001 0.001"/>
     </geometry>
   </collision>
@@ -93,5 +93,5 @@
     <origin rpy="0 0 0" xyz="0.271362 -0.354601 -0.057401"/>
     <geometry>
-      <mesh filename="package://v6_description/meshes/new_motor_v2_1.stl" scale="0.001 0.001 0.001"/>
+      <mesh filename="v6_description/meshes/new_motor_v2_1.stl" scale="0.001 0.001 0.001"/>
     </geometry>
     <material name="silver"/>
@@ -100,5 +100,5 @@
     <origin rpy="0 0 0" xyz="0.271362 -0.354601 -0.057401"/>
     <geometry>
-      <mesh filename="package://v6_description/meshes/new_motor_v2_1.stl" scale="0.001 0.001 0.001"/>
+      <mesh filename="v6_description/meshes/new_motor_v2_1.stl" scale="0.001 0.001 0.001"/>
     </geometry>
   </collision>
@@ -113,5 +113,5 @@
     <origin rpy="0 0 0" xyz="0.034705 -0.234351 -0.052597"/>
     <geometry>
-      <mesh filename="package://v6_description/meshes/car_stand_v2_1.stl" scale="0.001 0.001 0.001"/>
+      <mesh filename="v6_description/meshes/car_stand_v2_1.stl" scale="0.001 0.001 0.001"/>
     </geometry>
     <material name="silver"/>
@@ -120,5 +120,5 @@
     <origin rpy="0 0 0" xyz="0.034705 -0.234351 -0.052597"/>
     <geometry>
-      <mesh filename="package://v6_description/meshes/car_stand_v2_1.stl" scale="0.001 0.001 0.001"/>
+      <mesh filename="v6_description/meshes/car_stand_v2_1.stl" scale="0.001 0.001 0.001"/>
     </geometry>
   </collision>
@@ -133,5 +133,5 @@
     <origin rpy="0 0 0" xyz="-0.038906 -0.234351 -0.017587"/>
     <geometry>
-      <mesh filename="package://v6_description/meshes/car_stand_2_v2_v1_1.stl" scale="0.001 0.001 0.001"/>
+      <mesh filename="v6_description/meshes/car_stand_2_v2_v1_1.stl" scale="0.001 0.001 0.001"/>
     </geometry>
     <material name="silver"/>
@@ -140,5 +140,5 @@
     <origin rpy="0 0 0" xyz="-0.038906 -0.234351 -0.017587"/>
     <geometry>
-      <mesh filename="package://v6_description/meshes/car_stand_2_v2_v1_1.stl" scale="0.001 0.001 0.001"/>
+      <mesh filename="v6_description/meshes/car_stand_2_v2_v1_1.stl" scale="0.001 0.001 0.001"/>
     </geometry>
   </collision>
@@ -153,5 +153,5 @@
     <origin rpy="0 0 0" xyz="-0.030068 -0.229351 -0.008748"/>
     <geometry>
-      <mesh filename="package://v6_description/meshes/new_wheel_v1_1.stl" scale="0.001 0.001 0.001"/>
+      <mesh filename="v6_description/meshes/new_wheel_v1_1.stl" scale="0.001 0.001 0.001"/>
     </geometry>
     <material name="silver"/>
@@ -160,5 +160,5 @@
     <origin rpy="0 0 0" xyz="-0.030068 -0.229351 -0.008748"/>
     <geometry>
-      <mesh filename="package://v6_description/meshes/new_wheel_v1_1.stl" scale="0.001 0.001 0.001"/>
+      <mesh filename="v6_description/meshes/new_wheel_v1_1.stl" scale="0.001 0.001 0.001"/>
     </geometry>
   </collision>
@@ -173,5 +173,5 @@
     <origin rpy="0 0 0" xyz="0.034705 -0.434351 -0.052597"/>
     <geometry>
-      <mesh filename="package://v6_description/meshes/car_stand_v2__1__1.stl" scale="0.001 0.001 0.001"/>
+      <mesh filename="v6_description/meshes/car_stand_v2__1__1.stl" scale="0.001 0.001 0.001"/>
     </geometry>
     <material name="silver"/>
@@ -180,5 +180,5 @@
     <origin rpy="0 0 0" xyz="0.034705 -0.434351 -0.052597"/>
     <geometry>
-      <mesh filename="package://v6_description/meshes/car_stand_v2__1__1.stl" scale="0.001 0.001 0.001"/>
+      <mesh filename="v6_description/meshes/car_stand_v2__1__1.stl" scale="0.001 0.001 0.001"/>
     </geometry>
   </collision>
@@ -193,5 +193,5 @@
     <origin rpy="0 0 0" xyz="-0.038906 -0.434351 -0.017587"/>
     <geometry>
-      <mesh filename="package://v6_description/meshes/car_stand_2_v2_v1__1__1.stl" scale="0.001 0.001 0.001"/>
+      <mesh filename="v6_description/meshes/car_stand_2_v2_v1__1__1.stl" scale="0.001 0.001 0.001"/>
     </geometry>
     <material name="silver"/>
@@ -200,5 +200,5 @@
     <origin rpy="0 0 0" xyz="-0.038906 -0.434351 -0.017587"/>
     <geometry>
-      <mesh filename="package://v6_description/meshes/car_stand_2_v2_v1__1__1.stl" scale="0.001 0.001 0.001"/>
+      <mesh filename="v6_description/meshes/car_stand_2_v2_v1__1__1.stl" scale="0.001 0.001 0.001"/>
     </geometry>
   </collision>
@@ -213,5 +213,5 @@
     <origin rpy="0 0 0" xyz="-0.030068 -0.439351 -0.008748"/>
     <geometry>
-      <mesh filename="package://v6_description/meshes/new_wheel_v1__1__1.stl" scale="0.001 0.001 0.001"/>
+      <mesh filename="v6_description/meshes/new_wheel_v1__1__1.stl" scale="0.001 0.001 0.001"/>
     </geometry>
     <material name="silver"/>
@@ -220,5 +220,5 @@
     <origin rpy="0 0 0" xyz="-0.030068 -0.439351 -0.008748"/>
     <geometry>
-      <mesh filename="package://v6_description/meshes/new_wheel_v1__1__1.stl" scale="0.001 0.001 0.001"/>
+      <mesh filename="v6_description/meshes/new_wheel_v1__1__1.stl" scale="0.001 0.001 0.001"/>
     </geometry>
   </collision>
@@ -233,5 +233,5 @@
     <origin rpy="0 0 0" xyz="0.193373 -0.234351 -0.052597"/>
     <geometry>
-      <mesh filename="package://v6_description/meshes/car_stand_v2__2__1.stl" scale="0.001 0.001 0.001"/>
+      <mesh filename="v6_description/meshes/car_stand_v2__2__1.stl" scale="0.001 0.001 0.001"/>
     </geometry>
     <material name="silver"/>
@@ -240,5 +240,5 @@
     <origin rpy="0 0 0" xyz="0.193373 -0.234351 -0.052597"/>
     <geometry>
-      <mesh filename="package://v6_description/meshes/car_stand_v2__2__1.stl" scale="0.001 0.001 0.001"/>
+      <mesh filename="v6_description/meshes/car_stand_v2__2__1.stl" scale="0.001 0.001 0.001"/>
     </geometry>
   </collision>
@@ -253,5 +253,5 @@
     <origin rpy="0 0 0" xyz="0.266985 -0.234351 -0.017587"/>
     <geometry>
-      <mesh filename="package://v6_description/meshes/car_stand_2_v2_v1__2__1.stl" scale="0.001 0.001 0.001"/>
+      <mesh filename="v6_description/meshes/car_stand_2_v2_v1__2__1.stl" scale="0.001 0.001 0.001"/>
     </geometry>
     <material name="silver"/>
@@ -260,5 +260,5 @@
     <origin rpy="0 0 0" xyz="0.266985 -0.234351 -0.017587"/>
     <geometry>
-      <mesh filename="package://v6_description/meshes/car_stand_2_v2_v1__2__1.stl" scale="0.001 0.001 0.001"/>
+      <mesh filename="v6_description/meshes/car_stand_2_v2_v1__2__1.stl" scale="0.001 0.001 0.001"/>
     </geometry>
   </collision>
@@ -273,5 +273,5 @@
     <origin rpy="0 0 0" xyz="0.258146 -0.229351 -0.008748"/>
     <geometry>
-      <mesh filename="package://v6_description/meshes/new_wheel_v1__2__1.stl" scale="0.001 0.001 0.001"/>
+      <mesh filename="v6_description/meshes/new_wheel_v1__2__1.stl" scale="0.001 0.001 0.001"/>
     </geometry>
     <material name="silver"/>
@@ -280,5 +280,5 @@
     <origin rpy="0 0 0" xyz="0.258146 -0.229351 -0.008748"/>
     <geometry>
-      <mesh filename="package://v6_description/meshes/new_wheel_v1__2__1.stl" scale="0.001 0.001 0.001"/>
+      <mesh filename="v6_description/meshes/new_wheel_v1__2__1.stl" scale="0.001 0.001 0.001"/>
     </geometry>
   </collision>
@@ -293,5 +293,5 @@
     <origin rpy="0 0 0" xyz="0.209373 -0.434351 -0.052597"/>
     <geometry>
-      <mesh filename="package://v6_description/meshes/car_stand_v2__2___1__1.stl" scale="0.001 0.001 0.001"/>
+      <mesh filename="v6_description/meshes/car_stand_v2__2___1__1.stl" scale="0.001 0.001 0.001"/>
     </geometry>
     <material name="silver"/>
@@ -300,5 +300,5 @@
     <origin rpy="0 0 0" xyz="0.209373 -0.434351 -0.052597"/>
     <geometry>
-      <mesh filename="package://v6_description/meshes/car_stand_v2__2___1__1.stl" scale="0.001 0.001 0.001"/>
+      <mesh filename="v6_description/meshes/car_stand_v2__2___1__1.stl" scale="0.001 0.001 0.001"/>
     </geometry>
   </collision>
@@ -313,5 +313,5 @@
     <origin rpy="0 0 0" xyz="0.266985 -0.434351 -0.017587"/>
     <geometry>
-      <mesh filename="package://v6_description/meshes/car_stand_2_v2_v1__2___1__1.stl" scale="0.001 0.001 0.001"/>
+      <mesh filename="v6_description/meshes/car_stand_2_v2_v1__2___1__1.stl" scale="0.001 0.001 0.001"/>
     </geometry>
     <material name="silver"/>
@@ -320,5 +320,5 @@
     <origin rpy="0 0 0" xyz="0.266985 -0.434351 -0.017587"/>
     <geometry>
-      <mesh filename="package://v6_description/meshes/car_stand_2_v2_v1__2___1__1.stl" scale="0.001 0.001 0.001"/>
+      <mesh filename="v6_description/meshes/car_stand_2_v2_v1__2___1__1.stl" scale="0.001 0.001 0.001"/>
     </geometry>
   </collision>
@@ -333,5 +333,5 @@
     <origin rpy="0 0 0" xyz="0.258146 -0.439351 -0.008748"/>
     <geometry>
-      <mesh filename="package://v6_description/meshes/new_wheel_v1__2___1__1.stl" scale="0.001 0.001 0.001"/>
+      <mesh filename="v6_description/meshes/new_wheel_v1__2___1__1.stl" scale="0.001 0.001 0.001"/>
     </geometry>
     <material name="silver"/>
@@ -340,5 +340,5 @@
     <origin rpy="0 0 0" xyz="0.258146 -0.439351 -0.008748"/>
     <geometry>
-      <mesh filename="package://v6_description/meshes/new_wheel_v1__2___1__1.stl" scale="0.001 0.001 0.001"/>
+      <mesh filename="v6_description/meshes/new_wheel_v1__2___1__1.stl" scale="0.001 0.001 0.001"/>
     </geometry>
   </collision>
@@ -346,12 +346,12 @@
 <link name="big_U_self_v2_1">
   <inertial>
-    <origin rpy="0 0 0" xyz="-0.02423767526178927 -8.991950056769227e-08 -8.853660350069403e-06"/>
+    <origin rpy="0 0 0" xyz="-9.161679706937154e-06 -8.991395844537564e-08 0.024237580500525185"/>
     <mass value="0.041847447766480805"/>
-    <inertia ixx="2.4e-05" ixy="0.0" ixz="-0.0" iyy="1.1e-05" iyz="-0.0" izz="3.2e-05"/>
+    <inertia ixx="3.2e-05" ixy="0.0" ixz="0.0" iyy="1.1e-05" iyz="0.0" izz="2.4e-05"/>
   </inertial>
   <visual>
     <origin rpy="0 0 0" xyz="0.278674 -0.334851 -0.085006"/>
     <geometry>
-      <mesh filename="package://v6_description/meshes/big_U_self_v2_1.stl" scale="0.001 0.001 0.001"/>
+      <mesh filename="v6_description/meshes/big_U_self_v2_1.stl" scale="0.001 0.001 0.001"/>
     </geometry>
     <material name="silver"/>
@@ -360,5 +360,5 @@
     <origin rpy="0 0 0" xyz="0.278674 -0.334851 -0.085006"/>
     <geometry>
-      <mesh filename="package://v6_description/meshes/big_U_self_v2_1.stl" scale="0.001 0.001 0.001"/>
+      <mesh filename="v6_description/meshes/big_U_self_v2_1.stl" scale="0.001 0.001 0.001"/>
     </geometry>
   </collision>
@@ -366,19 +366,19 @@
 <link name="small_U_self_v3_v2_1">
   <inertial>
-    <origin rpy="0 0 0" xyz="-0.009287648733685094 -0.0005384482220820441 -3.1143207411127305e-06"/>
+    <origin rpy="0 0 0" xyz="-3.4223399267285792e-06 -0.0005384482108122812 0.009287553972544299"/>
     <mass value="0.025534175468152884"/>
-    <inertia ixx="9e-06" ixy="-0.0" ixz="-0.0" iyy="3e-06" iyz="-0.0" izz="1e-05"/>
-  </inertial>
-  <visual>
-    <origin rpy="0 0 0" xyz="0.318674 -0.334851 -0.084991"/>
-    <geometry>
-      <mesh filename="package://v6_description/meshes/small_U_self_v3_v2_1.stl" scale="0.001 0.001 0.001"/>
-    </geometry>
-    <material name="silver"/>
-  </visual>
-  <collision>
-    <origin rpy="0 0 0" xyz="0.318674 -0.334851 -0.084991"/>
-    <geometry>
-      <mesh filename="package://v6_description/meshes/small_U_self_v3_v2_1.stl" scale="0.001 0.001 0.001"/>
+    <inertia ixx="1e-05" ixy="-0.0" ixz="0.0" iyy="3e-06" iyz="0.0" izz="9e-06"/>
+  </inertial>
+  <visual>
+    <origin rpy="0 0 0" xyz="0.278689 -0.334851 -0.125006"/>
+    <geometry>
+      <mesh filename="v6_description/meshes/small_U_self_v3_v2_1.stl" scale="0.001 0.001 0.001"/>
+    </geometry>
+    <material name="silver"/>
+  </visual>
+  <collision>
+    <origin rpy="0 0 0" xyz="0.278689 -0.334851 -0.125006"/>
+    <geometry>
+      <mesh filename="v6_description/meshes/small_U_self_v3_v2_1.stl" scale="0.001 0.001 0.001"/>
     </geometry>
   </collision>
@@ -386,19 +386,19 @@
 <link name="new_motor_v2__1__1">
   <inertial>
-    <origin rpy="0 0 0" xyz="-0.0026535935407322464 0.02242666042984809 -0.007555050277332054"/>
+    <origin rpy="0 0 0" xyz="-0.007555358297381132 0.02242666044587277 0.002653498778970337"/>
     <mass value="0.20364393858439991"/>
-    <inertia ixx="3e-05" ixy="-0.0" ixz="-0.0" iyy="3.5e-05" iyz="-0.0" izz="5.1e-05"/>
-  </inertial>
-  <visual>
-    <origin rpy="0 0 0" xyz="0.346177 -0.314601 -0.092481"/>
-    <geometry>
-      <mesh filename="package://v6_description/meshes/new_motor_v2__1__1.stl" scale="0.001 0.001 0.001"/>
-    </geometry>
-    <material name="silver"/>
-  </visual>
-  <collision>
-    <origin rpy="0 0 0" xyz="0.346177 -0.314601 -0.092481"/>
-    <geometry>
-      <mesh filename="package://v6_description/meshes/new_motor_v2__1__1.stl" scale="0.001 0.001 0.001"/>
+    <inertia ixx="5.1e-05" ixy="-0.0" ixz="0.0" iyy="3.5e-05" iyz="0.0" izz="3e-05"/>
+  </inertial>
+  <visual>
+    <origin rpy="0 0 0" xyz="0.271199 -0.314601 -0.152509"/>
+    <geometry>
+      <mesh filename="v6_description/meshes/new_motor_v2__1__1.stl" scale="0.001 0.001 0.001"/>
+    </geometry>
+    <material name="silver"/>
+  </visual>
+  <collision>
+    <origin rpy="0 0 0" xyz="0.271199 -0.314601 -0.152509"/>
+    <geometry>
+      <mesh filename="v6_description/meshes/new_motor_v2__1__1.stl" scale="0.001 0.001 0.001"/>
     </geometry>
   </collision>
@@ -406,19 +406,19 @@
 <link name="big_U_self_v2__1__1">
   <inertial>
-    <origin rpy="0 0 0" xyz="-9.12643416350889e-06 -8.993477979002407e-08 0.024237117404991515"/>
+    <origin rpy="0 0 0" xyz="0.020995083755278143 -8.99093536843587e-08 -0.01211090571389134"/>
     <mass value="0.04184744776647988"/>
-    <inertia ixx="3.2e-05" ixy="0.0" ixz="0.0" iyy="1.1e-05" iyz="-0.0" izz="2.4e-05"/>
-  </inertial>
-  <visual>
-    <origin rpy="0 0 0" xyz="0.358674 -0.334351 -0.084977"/>
-    <geometry>
-      <mesh filename="package://v6_description/meshes/big_U_self_v2__1__1.stl" scale="0.001 0.001 0.001"/>
-    </geometry>
-    <material name="silver"/>
-  </visual>
-  <collision>
-    <origin rpy="0 0 0" xyz="0.358674 -0.334351 -0.084977"/>
-    <geometry>
-      <mesh filename="package://v6_description/meshes/big_U_self_v2__1__1.stl" scale="0.001 0.001 0.001"/>
+    <inertia ixx="2.6e-05" ixy="0.0" ixz="4e-06" iyy="1.1e-05" iyz="0.0" izz="3e-05"/>
+  </inertial>
+  <visual>
+    <origin rpy="0 0 0" xyz="0.278704 -0.334351 -0.165006"/>
+    <geometry>
+      <mesh filename="v6_description/meshes/big_U_self_v2__1__1.stl" scale="0.001 0.001 0.001"/>
+    </geometry>
+    <material name="silver"/>
+  </visual>
+  <collision>
+    <origin rpy="0 0 0" xyz="0.278704 -0.334351 -0.165006"/>
+    <geometry>
+      <mesh filename="v6_description/meshes/big_U_self_v2__1__1.stl" scale="0.001 0.001 0.001"/>
     </geometry>
   </collision>
@@ -426,19 +426,19 @@
 <link name="grap_base_v1_1">
   <inertial>
-    <origin rpy="0 0 0" xyz="5.0604957804400996e-05 -8.993024042114328e-08 0.01574867865416396"/>
+    <origin rpy="0 0 0" xyz="0.013613530613986763 -8.989555810856587e-08 -0.007918424860268225"/>
     <mass value="0.16096668074514336"/>
-    <inertia ixx="6.6e-05" ixy="-0.0" ixz="-0.0" iyy="9.8e-05" iyz="-0.0" izz="9.8e-05"/>
-  </inertial>
-  <visual>
-    <origin rpy="0 0 0" xyz="0.358689 -0.334351 -0.124977"/>
-    <geometry>
-      <mesh filename="package://v6_description/meshes/grap_base_v1_1.stl" scale="0.001 0.001 0.001"/>
-    </geometry>
-    <material name="silver"/>
-  </visual>
-  <collision>
-    <origin rpy="0 0 0" xyz="0.358689 -0.334351 -0.124977"/>
-    <geometry>
-      <mesh filename="package://v6_description/meshes/grap_base_v1_1.stl" scale="0.001 0.001 0.001"/>
+    <inertia ixx="9e-05" ixy="-0.0" ixz="-1.4e-05" iyy="9.8e-05" iyz="-0.0" izz="7.4e-05"/>
+  </inertial>
+  <visual>
+    <origin rpy="0 0 0" xyz="0.244055 -0.334351 -0.145019"/>
+    <geometry>
+      <mesh filename="v6_description/meshes/grap_base_v1_1.stl" scale="0.001 0.001 0.001"/>
+    </geometry>
+    <material name="silver"/>
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