Commit message: Update mac_car

File: mac_car/v6_description/v6_unity_urdf/v6.urdf (robot description, URDF)
Before this commit: robot v6, 24 links, 23 joints
Links:
- added link LiDAR_v1_1, mass 0.31975775721502164; collision mesh filename=v6_description/meshes/LiDAR_v1_1.stl scale=0.001 0.001 0.001; visual mesh filename=v6_description/meshes/LiDAR_v1_1.stl scale=0.001 0.001 0.001
- added link camera_1, mass 0.2435559840000003; collision mesh filename=v6_description/meshes/camera_1.stl scale=0.001 0.001 0.001; visual mesh filename=v6_description/meshes/camera_1.stl scale=0.001 0.001 0.001
- added link camera_support_1, mass 0.04003969304541568; collision mesh filename=v6_description/meshes/camera_support_1.stl scale=0.001 0.001 0.001; visual mesh filename=v6_description/meshes/camera_support_1.stl scale=0.001 0.001 0.001
- link Side_U_Bracket_Component1_v2_1: geometry collision mesh filename=v6_description/meshes/Side_U_Bracket_Component1_v2_1.stl scale=0.001 0.001 0.001; visual mesh filename=v6_description/meshes/Side_U_Bracket_Component1_v2_1.stl scale=0.001 0.001 0.001
- link base_link: geometry collision mesh filename=v6_description/meshes/base_link.stl scale=0.001 0.001 0.001; visual mesh filename=v6_description/meshes/base_link.stl scale=0.001 0.001 0.001
- link big_U_self_v2_1: geometry collision mesh filename=v6_description/meshes/big_U_self_v2_1.stl scale=0.001 0.001 0.001; visual mesh filename=v6_description/meshes/big_U_self_v2_1.stl scale=0.001 0.001 0.001
- link big_U_self_v2__1__1: geometry collision mesh filename=v6_description/meshes/big_U_self_v2__1__1.stl scale=0.001 0.001 0.001; visual mesh filename=v6_description/meshes/big_U_self_v2__1__1.stl scale=0.001 0.001 0.001
- link car_stand_2_v2_v1_1: geometry collision mesh filename=v6_description/meshes/car_stand_2_v2_v1_1.stl scale=0.001 0.001 0.001; visual mesh filename=v6_description/meshes/car_stand_2_v2_v1_1.stl scale=0.001 0.001 0.001
- link car_stand_2_v2_v1__1__1: geometry collision mesh filename=v6_description/meshes/car_stand_2_v2_v1__1__1.stl scale=0.001 0.001 0.001; visual mesh filename=v6_description/meshes/car_stand_2_v2_v1__1__1.stl scale=0.001 0.001 0.001
- link car_stand_2_v2_v1__2__1: geometry collision mesh filename=v6_description/meshes/car_stand_2_v2_v1__2__1.stl scale=0.001 0.001 0.001; visual mesh filename=v6_description/meshes/car_stand_2_v2_v1__2__1.stl scale=0.001 0.001 0.001
- link car_stand_2_v2_v1__2___1__1: geometry collision mesh filename=v6_description/meshes/car_stand_2_v2_v1__2___1__1.stl scale=0.001 0.001 0.001; visual mesh filename=v6_description/meshes/car_stand_2_v2_v1__2___1__1.stl scale=0.001 0.001 0.001
- link car_stand_v2_1: geometry collision mesh filename=v6_description/meshes/car_stand_v2_1.stl scale=0.001 0.001 0.001; visual mesh filename=v6_description/meshes/car_stand_v2_1.stl scale=0.001 0.001 0.001
- link car_stand_v2__1__1: geometry collision mesh filename=v6_description/meshes/car_stand_v2__1__1.stl scale=0.001 0.001 0.001; visual mesh filename=v6_description/meshes/car_stand_v2__1__1.stl scale=0.001 0.001 0.001
- link car_stand_v2__2__1: geometry collision mesh filename=v6_description/meshes/car_stand_v2__2__1.stl scale=0.001 0.001 0.001; visual mesh filename=v6_description/meshes/car_stand_v2__2__1.stl scale=0.001 0.001 0.001
- link car_stand_v2__2___1__1: geometry collision mesh filename=v6_description/meshes/car_stand_v2__2___1__1.stl scale=0.001 0.001 0.001; visual mesh filename=v6_description/meshes/car_stand_v2__2___1__1.stl scale=0.001 0.001 0.001
- link grap2_v2_1: geometry collision mesh filename=v6_description/meshes/grap2_v2_1.stl scale=0.001 0.001 0.001; visual mesh filename=v6_description/meshes/grap2_v2_1.stl scale=0.001 0.001 0.001
- link grap2_v2_Mirror__1: geometry collision mesh filename=v6_description/meshes/grap2_v2_Mirror__1.stl scale=0.001 0.001 0.001; visual mesh filename=v6_description/meshes/grap2_v2_Mirror__1.stl scale=0.001 0.001 0.001
- link grap_base_v1_1: geometry collision mesh filename=v6_description/meshes/grap_base_v1_1.stl scale=0.001 0.001 0.001; visual mesh filename=v6_description/meshes/grap_base_v1_1.stl scale=0.001 0.001 0.001
- link new_motor_v2_1: geometry collision mesh filename=v6_description/meshes/new_motor_v2_1.stl scale=0.001 0.001 0.001; visual mesh filename=v6_description/meshes/new_motor_v2_1.stl scale=0.001 0.001 0.001
- link new_motor_v2__1__1: geometry collision mesh filename=v6_description/meshes/new_motor_v2__1__1.stl scale=0.001 0.001 0.001; visual mesh filename=v6_description/meshes/new_motor_v2__1__1.stl scale=0.001 0.001 0.001
- link new_wheel_v1_1: geometry collision mesh filename=v6_description/meshes/new_wheel_v1_1.stl scale=0.001 0.001 0.001; visual mesh filename=v6_description/meshes/new_wheel_v1_1.stl scale=0.001 0.001 0.001
- link new_wheel_v1__1__1: geometry collision mesh filename=v6_description/meshes/new_wheel_v1__1__1.stl scale=0.001 0.001 0.001; visual mesh filename=v6_description/meshes/new_wheel_v1__1__1.stl scale=0.001 0.001 0.001
- link new_wheel_v1__2__1: geometry collision mesh filename=v6_description/meshes/new_wheel_v1__2__1.stl scale=0.001 0.001 0.001; visual mesh filename=v6_description/meshes/new_wheel_v1__2__1.stl scale=0.001 0.001 0.001
- link new_wheel_v1__2___1__1: geometry collision mesh filename=v6_description/meshes/new_wheel_v1__2___1__1.stl scale=0.001 0.001 0.001; visual mesh filename=v6_description/meshes/new_wheel_v1__2___1__1.stl scale=0.001 0.001 0.001
- link small_U_self_v3_v2_1: geometry collision mesh filename=v6_description/meshes/small_U_self_v3_v2_1.stl scale=0.001 0.001 0.001; visual mesh filename=v6_description/meshes/small_U_self_v3_v2_1.stl scale=0.001 0.001 0.001
- link upper_blue_v1_1: geometry collision mesh filename=v6_description/meshes/upper_blue_v1_1.stl scale=0.001 0.001 0.001; visual mesh filename=v6_description/meshes/upper_blue_v1_1.stl scale=0.001 0.001 0.001
- link upper_silver_v1_1: mass 0.5824308278195107 -> 0.5901067825147455; geometry collision mesh filename=v6_description/meshes/upper_silver_v1_1.stl scale=0.001 0.001 0.001; visual mesh filename=v6_description/meshes/upper_silver_v1_1.stl scale=0.001 0.001 0.001
Joints:
- added joint Revolute 51: type continuous, parent upper_silver_v1_1, child camera_support_1, origin xyz=-0.088244 0.128656 0.095323 rpy=0 0 0, axis -0.0 -1.0 -0.0
- added joint Rigid 50: type fixed, parent upper_silver_v1_1, child LiDAR_v1_1, origin xyz=-0.050498 0.128656 0.106268 rpy=0 0 0
- added joint Rigid 52: type fixed, parent camera_support_1, child camera_1, origin xyz=0.001192 0.0 0.022082 rpy=0 0 0
- joint Revolute 44: origin xyz=-0.012497 0.01975 -0.007504 rpy=0 0 0 -> xyz=-0.007505 0.01975 0.012497 rpy=0 0 0
- joint Revolute 48: axis -1.0 -0.0 -0.00037 -> 0.49968 0.0 0.86621; origin xyz=-1.3e-05 0.0125 0.0355 rpy=0 0 0 -> xyz=0.03075 0.0125 -0.017739 rpy=0 0 0
- joint Revolute 49: axis 1.0 0.0 0.00037 -> -0.49968 -0.0 -0.86621; origin xyz=-1.3e-05 -0.0125 0.0355 rpy=0 0 0 -> xyz=0.03075 -0.0125 -0.017739 rpy=0 0 0
- joint Rigid 42: origin xyz=-0.04 0.0 -1.5e-05 rpy=0 0 0 -> xyz=-1.5e-05 0.0 0.04 rpy=0 0 0
- joint Rigid 43: origin xyz=-0.027503 -0.02025 0.00749 rpy=0 0 0 -> xyz=0.00749 -0.02025 0.027503 rpy=0 0 0
- joint Rigid 45: origin xyz=-1.5e-05 0.0 0.04 rpy=0 0 0 -> xyz=0.034649 0.0 -0.019987 rpy=0 0 0
